File: Boards/BMS_Data_Acquisition/DA_Board_1/DA_Board_1.kicad_pcb (KiCad board)
At the start: 2 copper layers, 490.8 x 272 mm, 91 parts, among them J1 MM_F_VT_12, J1 MM_M_VT_10, J10 MM_F_VT_04, J2 MM_F_VT_10, J2 MM_M_VT_12, J3 MM_F_VT_16, J3 MM_M_VT_12, J4 MM_F_VT_12, J4 MM_M_VT_12, J5 MM_M_VT_12, J5 MM_M_VT_16, J6 MM_M_VT_10, J7 MM_M_VT_12, J8 MM_F_VT_04, J8 MM_M_VT_12, J9 MM_M_VT_12, Q10 BSS308PE, Q12 BSS308PE, Q14 BSS308PE, Q16 BSS308PE, Q2 BSS308PE, Q4 BSS308PE, Q6 BSS308PE, Q8 BSS308PE, T0 Tab_Connect_BMS, T10 Tab_Connect_BMS, T12 Tab_Connect_BMS, T14 Tab_Connect_BMS, T16 Tab_Connect_BMS, T2 Tab_Connect_BMS, T4 Tab_Connect_BMS, T6 Tab_Connect_BMS, T8 Tab_Connect_BMS

Commit message: slight changes for BMS boards before shipping
Parts:
- removed the J1 at (491.1, 253.9)
- removed the J2 at (490.0, 229.4)
- removed the J3 at (491.3, 195.3)
- removed the J4 at (491.5, 171.4)
- removed the J5 at (491.5, 146.5)
- removed the J8 at (519.0, 365.9)
Other:
- board size 490.8 x 272 mm -> 340.1 x 60.8 mm
- board text added: "BMS Data Acquisition #1 Rev 2.0 Olin Electric Motorsports 2/27/2020 Vienna Scheyer '21, Wesley Soo-Hoo '23"
- board text removed: "BMS Data Acquisition #1 Rev 1.0 Olin Electric Motorsports Vienna Scheyer '21, Wesley Soo-Hoo '23"
Changed lines of the file:
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@@
-(kicad_pcb (version 20171130) (host pcbnew 5.1.5)
+(kicad_pcb (version 20171130) (host pcbnew 5.1.5-52549c5~84~ubuntu18.04.1)
   (general
     (thickness 1.6)
-    (drawings 84)
+    (drawings 76)
     (tracks 1658)
     (zones 0)
-    (modules 91)
+    (modules 85)
     (nets 117)
   )
@@
   )
   (setup
-    (last_trace_width 0.762)
+    (last_trace_width 0.254)
     (user_trace_width 0.254)
     (user_trace_width 0.381)
@@
     (pcbplotparams
       (layerselection 0x010fc_ffffffff)
-      (usegerberextensions false)
+      (usegerberextensions true)
       (usegerberattributes false)
       (usegerberadvancedattributes false)
@@
     )
   )
-  (module footprints:micromatch_female_vt_12 (layer B.Cu)
-    (at 491.49 146.5072 180)
-    (fp_text reference J5 (at 5.4404 -11.2608) (layer F.SilkS)
-      (effects (font (size 1 1) (thickness 0.15)))
-    )
-    (fp_text value MM_M_VT_12 (at 6.35 0 270) (layer B.Fab) hide
-      (effects (font (size 1 1) (thickness 0.15)) (justify mirror))
-    )
-    (fp_line (start 3.92 -11.83) (end 3.92 8.02) (layer B.SilkS) (width 0.15))
-    (fp_line (start -1.38 -11.83) (end -1.38 8.02) (layer B.SilkS) (width 0.15))
-    (fp_line (start -1.38 8.02) (end 3.92 8.02) (layer B.SilkS) (width 0.15))
-    (fp_line (start -1.38 -11.83) (end 3.92 -11.83) (layer B.SilkS) (width 0.15))
-    (fp_text user 1 (at 0 8.89) (layer F.SilkS)
-      (effects (font (size 1 1) (thickness 0.15)))
-    )
-    (fp_text user 12 (at 2.54 -12.7) (layer F.SilkS)
-      (effects (font (size 1 1) (thickness 0.15)))
-    )
-  )
-  (module footprints:micromatch_female_vert_16 (layer B.Cu)
-    (at 491.3376 195.326 180)
-    (fp_text reference J3 (at 5.688 -16.152) (layer F.SilkS)
-      (effects (font (size 1 1) (thickness 0.15)))
-    )
-    (fp_text value MM_F_VT_16 (at 6.35 0 270) (layer B.Fab) hide
-      (effects (font (size 1 1) (thickness 0.15)) (justify mirror))
-    )
-    (fp_line (start 3.92 -16.91) (end 3.92 8.02) (layer B.SilkS) (width 0.15))
-    (fp_line (start -1.38 -16.91) (end -1.38 8.02) (layer B.SilkS) (width 0.15))
-    (fp_line (start -1.38 8.02) (end 3.92 8.02) (layer B.SilkS) (width 0.15))
-    (fp_line (start -1.38 -16.91) (end 3.92 -16.91) (layer B.SilkS) (width 0.15))
-    (fp_text user 1 (at 0 8.89) (layer F.SilkS)
-      (effects (font (size 1 1) (thickness 0.15)))
-    )
-    (fp_text user 16 (at 2.54 -17.78) (layer F.SilkS)
-      (effects (font (size 1 1) (thickness 0.15)))
-    )
-  )
-  (module footprints:micromatch_female_vt_12 (layer B.Cu)
-    (at 491.49 171.3992 180)
-    (fp_text reference J4 (at 5.4404 -11.1388) (layer F.SilkS)
-      (effects (font (size 1 1) (thickness 0.15)))
-    )
-    (fp_text value MM_F_VT_12 (at 6.35 0 270) (layer B.Fab) hide
-      (effects (font (size 1 1) (thickness 0.15)) (justify mirror))
-    )
-    (fp_text user 12 (at 2.54 -12.7) (layer F.SilkS)
-      (effects (font (size 1 1) (thickness 0.15)))
-    )
-    (fp_text user 1 (at 0 8.89) (layer F.SilkS)
-      (effects (font (size 1 1) (thickness 0.15)))
-    )
-    (fp_line (start -1.38 -11.83) (end 3.92 -11.83) (layer B.SilkS) (width 0.15))
-    (fp_line (start -1.38 8.02) (end 3.92 8.02) (layer B.SilkS) (width 0.15))
-    (fp_line (start -1.38 -11.83) (end -1.38 8.02) (layer B.SilkS) (width 0.15))
-    (fp_line (start 3.92 -11.83) (end 3.92 8.02) (layer B.SilkS) (width 0.15))
-  )
-  (module footprints:micromatch_female_vt_12 (layer B.Cu)
-    (at 491.109 253.9492 180)
-    (fp_text reference J1 (at 5.3294 -11.1688) (layer F.SilkS)
-      (effects (font (size 1 1) (thickness 0.15)))
-    )
-    (fp_text value MM_F_VT_12 (at 6.35 0 270) (layer B.Fab) hide
-      (effects (font (size 1 1) (thickness 0.15)) (justify mirror))
-    )
-    (fp_line (start 3.92 -11.83) (end 3.92 8.02) (layer B.SilkS) (width 0.15))
-    (fp_line (start -1.38 -11.83) (end -1.38 8.02) (layer B.SilkS) (width 0.15))
-    (fp_line (start -1.38 8.02) (end 3.92 8.02) (layer B.SilkS) (width 0.15))
-    (fp_line (start -1.38 -11.83) (end 3.92 -11.83) (layer B.SilkS) (width 0.15))
-    (fp_text user 1 (at 0 8.89) (layer F.SilkS)
-      (effects (font (size 1 1) (thickness 0.15)))
-    )
-    (fp_text user 12 (at 2.7432 -13.0302) (layer F.SilkS)
-      (effects (font (size 1 1) (thickness 0.15)))
-    )
-  )
-  (module footprints:micromatch_female_vert_10 (layer B.Cu)
-    (at 490.0168 229.4382 180)
-    (fp_text reference J2 (at 4.3072 -8.3598) (layer F.SilkS)
-      (effects (font (size 1 1) (thickness 0.15)))
-    )
-    (fp_text value MM_F_VT_10 (at 5.1308 0.3048 270) (layer B.Fab) hide
-      (effects (font (size 1 1) (thickness 0.15)) (justify mirror))
-    )
-    (fp_line (start 2.65 -8.655) (end 2.65 8.655) (layer B.SilkS) (width 0.15))
-    (fp_line (start -2.65 -8.655) (end -2.65 8.655) (layer B.SilkS) (width 0.15))
-    (fp_line (start -2.65 8.655) (end 2.65 8.655) (layer B.SilkS) (width 0.15))
-    (fp_line (start -2.65 -8.655) (end 2.65 -8.655) (layer B.SilkS) (width 0.15))
-    (fp_text user 1 (at -1.27 9.525) (layer F.SilkS)
-      (effects (font (size 1 1) (thickness 0.15)))
-    )
-    (fp_text user 10 (at 1.27 -9.525) (layer F.SilkS)
-      (effects (font (size 1 1) (thickness 0.15)))
-    )
-  )
-  (module footprints:micromatch_female_vert_4 (layer B.Cu)
-    (at 518.9982 365.9378 270)
-    (fp_text reference J8 (at 5.08 0 270) (layer B.SilkS)
-      (effects (font (size 1 1) (thickness 0.15)) (justify mirror))
-    )
-    (fp_text value MM_F_VT_04 (at 6.35 1.27) (layer B.Fab) hide
-      (effects (font (size 1 1) (thickness 0.15)) (justify mirror))
-    )
-    (fp_text user 4 (at 2.54 -2.54 270) (layer B.SilkS)
-      (effects (font (size 1 1) (thickness 0.15)) (justify mirror))
-    )
-    (fp_text user 1 (at 0 8.89 270) (layer B.SilkS)
-      (effects (font (size 1 1) (thickness 0.15)) (justify mirror))
-    )
-    (fp_line (start -1.38 -1.67) (end 3.92 -1.67) (layer B.SilkS) (width 0.15))
-    (fp_line (start -1.38 8.02) (end 3.92 8.02) (layer B.SilkS) (width 0.15))
-    (fp_line (start -1.38 -1.67) (end -1.38 8.02) (layer B.SilkS) (width 0.15))
-    (fp_line (start 3.92 -1.67) (end 3.92 8.02) (layer B.SilkS) (width 0.15))
-  )
   (gr_arc (start 327.554818 163.702977) (end 337.820493 158.823096) (angle -64.57549777) (layer Edge.Cuts) (width 0.2))
   (gr_arc (start 122.248 157.46) (end 119.380493 158.823096) (angle -64.57549777) (layer Edge.Cuts) (width 0.2))
@@
   (gr_line (start 97.250387 156.571) (end 97.250387 154.241477) (layer Edge.Cuts) (width 0.2))
   (gr_arc (start 78.56 157.46) (end 75.692493 158.823096) (angle -64.57549777) (layer Edge.Cuts) (width 0.2))
-  (gr_text "BMS Data Acquisition #1 Rev 1.0\nOlin Electric Motorsports\nVienna Scheyer '21, Wesley Soo-Hoo '23" (at 214.4727 103.6576) (layer F.SilkS)
+  (gr_text "BMS Data Acquisition #1 Rev 2.0\nOlin Electric Motorsports\n2/27/2020\nVienna Scheyer '21, Wesley Soo-Hoo '23" (at 94.5896 107.8484) (layer F.SilkS)
     (effects (font (size 1.5 1.5) (thickness 0.3)))
   )
@@
   (gr_line (start 42.3418 149.856434) (end 272.211801 149.856434) (layer Dwgs.User) (width 0.2))
   (gr_line (start 39.1668 102.993434) (end 39.1668 146.681434) (layer Dwgs.User) (width 0.2))
-  (gr_arc (start 526.767034 368.681) (end 526.767034 371.856) (angle -90) (layer Edge.Cuts) (width 0.2))
-  (gr_line (start 526.767034 135.636) (end 483.079034 135.636) (layer Edge.Cuts) (width 0.2))
-  (gr_arc (start 483.079034 368.681) (end 479.904034 368.681) (angle -90) (layer Edge.Cuts) (width 0.2))
-  (gr_line (start 479.904034 138.810999) (end 479.904034 368.681) (layer Edge.Cuts) (width 0.2))
-  (gr_line (start 483.079034 371.856) (end 526.767034 371.856) (layer Edge.Cuts) (width 0.2))
-  (gr_line (start 529.942034 368.681) (end 529.942034 138.810999) (layer Edge.Cuts) (width 0.2))
-  (gr_arc (start 483.079034 138.810999) (end 483.079034 135.635999) (angle -90) (layer Edge.Cuts) (width 0.2))
-  (gr_arc (start 526.767034 138.810999) (end 529.942034 138.810999) (angle -90) (layer Edge.Cuts) (width 0.2))
   (segment (start 153.4746 146.0314) (end 152.4772 145.034) (width 0.254) (layer F.Cu) (net 1))
   (segment (start 153.4746 148.2854) (end 153.4746 146.0314) (width 0.254) (layer F.Cu) (net 1))
@@
       )
     )
+  )
+  (zone (net 0) (net_name "") (layer F.SilkS) (hatch full 0.508)
+    (connect_pads (clearance 0.508))
+    (min_thickness 0.254)
+    (fill yes (arc_segments 32) (thermal_gap 0.508) (thermal_bridge_width 0.508))
+    (polygon
+      (pts
+        (xy 114.808 129.9464) (xy 98.0186 129.9464) (xy 98.0186 116.9162) (xy 114.808 116.9162)
+      )
+    )
