File: Boards/BMS_Data_Acquisition/DA_Board_2/DA_Board_2.kicad_pcb (KiCad board)
At the start: 2 copper layers, 340.1 x 60.8 mm, 72 parts, among them J1 MM_M_VT_12, J2 MM_M_VT_12, J3 MM_M_VT_10, J4 MM_M_VT_12, Q1 BSS308PE, Q11 BSS308PE, Q13 BSS308PE, Q15 BSS308PE, Q3 BSS308PE, Q5 BSS308PE, Q7 BSS308PE, Q9 BSS308PE, T1 Tab_Connect_BMS, T11 Tab_Connect_BMS, T13 Tab_Connect_BMS, T15 Tab_Connect_BMS, T3 Tab_Connect_BMS, T5 Tab_Connect_BMS, T7 Tab_Connect_BMS, T9 Tab_Connect_BMS

Commit message: slight changes for BMS boards before shipping
Routing:
- added copper zone on B.Cu, net /GND1
Other:
- board text added: "BMS Data Acquisition #2 Rev 2.0 Olin Electric Motorsports 2/27/2020 Vienna Scheyer '21 Corey Cochran-Lepiz `21"
- board text removed: "BMS Data Acquisition #2 Rev 2.0 Olin Electric Motorsports Corey Cochran-Lepiz `21 Vienna Scheyer '21"
Changed lines of the file:
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@@
   )
   (setup
-    (last_trace_width 0.508)
+    (last_trace_width 0.25)
     (user_trace_width 0.254)
     (user_trace_width 0.508)
@@
     (pcbplotparams
       (layerselection 0x010fc_ffffffff)
-      (usegerberextensions false)
+      (usegerberextensions true)
       (usegerberattributes false)
       (usegerberadvancedattributes false)
@@
   (gr_line (start -19.474001 140.841458) (end 29.04 140.841458) (layer Edge.Cuts) (width 0.2))
   (gr_arc (start 29.04 152.13) (end 35.9096 143.172334) (angle -37.48446236) (layer Edge.Cuts) (width 0.2))
-  (gr_text "BMS Data Acquisition #2 Rev 2.0\nOlin Electric Motorsports\nCorey Cochran-Lepiz `21\nVienna Scheyer '21" (at 144.5006 99.3902) (layer F.SilkS)
+  (gr_text "BMS Data Acquisition #2 Rev 2.0\nOlin Electric Motorsports\n2/27/2020\nVienna Scheyer '21\nCorey Cochran-Lepiz `21" (at 144.5006 99.3902) (layer F.SilkS)
     (effects (font (size 1.5 1.5) (thickness 0.3)))
   )
@@
       )
     )
+  )
+  (zone (net 55) (net_name /GND1) (layer B.Cu) (hatch edge 0.508)
+    (connect_pads (clearance 0.508))
+    (min_thickness 0.254)
+    (fill yes (arc_segments 32) (thermal_gap 0.508) (thermal_bridge_width 0.508))
+    (polygon
+      (pts
+        (xy 323.7484 152.019) (xy -31.115 152.019) (xy -31.115 83.82) (xy 323.7484 83.82)
+      )
+    )
+  )
+  (zone (net 0) (net_name "") (layer F.SilkS) (hatch edge 0.508)
+    (connect_pads (clearance 0.508))
+    (min_thickness 0.254)
+    (fill yes (arc_segments 32) (thermal_gap 0.508) (thermal_bridge_width 0.508))
+    (polygon
+      (pts
+        (xy 181.991 105.6132) (xy 169.6212 105.6132) (xy 169.6212 94.8436) (xy 181.991 94.8436)
+      )
+    )
