File: Boards/BMS_Peripheral/BMS_peripheral.kicad_pcb (KiCad board)
At the start: 4 copper layers, 50 x 287 mm, 133 parts, among them J1 MM_F_VT_12, J2 MM_F_VT_10, J3 MM_F_VT_16, J4 MM_F_VT_12, J5 MM_M_VT_12, J6 MicroFit_RA_V_2_SMD, J7 MicroFit_RA_V_2_SMD, Q1 NSS1C201MZ4, Q2 NSS1C201MZ4, T1 T_LAN_SM91501ALE, T2 T_LAN_SM91501ALE, U1 LTC6811-1, U2 LTC6811-1, U3 24AA01, U4 MCP6001T-I-LT, U5 LTC1380IGN, U6 LTC1380IGN, U7 LTC1380IGN, U8 MCP6001T-I-LT

Commit message: slight changes for BMS boards before shipping
Parts:
- added ?: , , F.Cu at (182.9, 274.0)
- added J8: MM_F_VT_04, footprints:micromatch_female_vert_4, B.Cu at (213.6, 373.0)
- added TP1: Test_Point_SMD, footprints:Test_Point_SMD, F.Cu at (198.6, 351.9)
- added TP10: Test_Point_SMD, footprints:Test_Point_SMD, F.Cu at (198.7, 319.1)
- added TP11: Test_Point_SMD, footprints:Test_Point_SMD, F.Cu at (198.6, 347.8)
- added TP12: Test_Point_SMD, footprints:Test_Point_SMD, F.Cu at (198.6, 340.9)
- added TP13: Test_Point_SMD, footprints:Test_Point_SMD, F.Cu at (198.6, 332.9)
- added TP14: Test_Point_SMD, footprints:Test_Point_SMD, F.Cu at (198.6, 327.2)
- added TP2: Test_Point_SMD, footprints:Test_Point_SMD, F.Cu at (192.6, 287.1)
- added TP3: Test_Point_SMD, footprints:Test_Point_SMD, F.Cu at (193.7, 292.0)
- added TP4: Test_Point_SMD, footprints:Test_Point_SMD, F.Cu at (198.6, 355.7)
- added TP5: Test_Point_SMD, footprints:Test_Point_SMD, F.Cu at (221.8, 324.5)
- added TP6: Test_Point_SMD, footprints:Test_Point_SMD, F.Cu at (198.6, 359.3)
- added TP7: Test_Point_SMD, footprints:Test_Point_SMD, F.Cu at (206.2, 365.3)
- added TP8: Test_Point_SMD, footprints:Test_Point_SMD, F.Cu at (212.1, 321.3)
- added TP9: Test_Point_SMD, footprints:Test_Point_SMD, F.Cu at (198.7, 322.5)
- moved C1 203.9 mm to (218.7, 319.4), turned to 0 degrees
- moved C2 203.3 mm to (218.7, 317.3)
- moved C3 202.8 mm to (218.7, 315.1), turned to 0 degrees
- moved C4 202.4 mm to (218.7, 312.9)
- moved C5 202.1 mm to (218.7, 310.8), turned to 0 degrees
- moved C6 201.9 mm to (218.7, 308.6)
- moved C8 201.8 mm to (218.7, 304.3)
- moved C7 201.8 mm to (218.7, 306.4), turned to 0 degrees
- moved U1 179.7 mm to (209.8, 308.6), turned to 180 degrees
- moved R37 174.5 mm to (203.2, 315.2), turned to 90 degrees
- moved R40 171.5 mm to (200.9, 315.1), turned to 90 degrees
- moved C22 171.1 mm to (202.0, 312.2), turned to 180 degrees
- moved C24 170.3 mm to (188.1, 302.6), turned to 0 degrees
- moved C20 170.1 mm to (202.0, 310.1), turned to 180 degrees
- moved C19 169.1 mm to (202.0, 308.1), turned to 180 degrees
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Routing:
- net /VREF2: track 201.7 -> 457.9 mm, vias 0 -> 10
- net /C9: track 250.5 -> 25.2 mm, vias 2 -> 0
- net /C15: track 246.5 -> 21.8 mm, vias 2 -> 0
- net /C13: track 246.4 -> 22.5 mm, vias 2 -> 0
- net Net-(C14-Pad2): track 16.5 -> 239.4 mm, vias 0 -> 3
- net /C4: track 246.4 -> 24.0 mm, vias 3 -> 0
- net /C2: track 242.0 -> 21.9 mm, vias 2 -> 0
- net /C11: track 243.2 -> 24.3 mm, vias 2 -> 0
- net Net-(C12-Pad2): track 21.7 -> 239.9 mm, vias 0 -> 3
- net Net-(C10-Pad2): track 18.0 -> 235.5 mm, vias 0 -> 3
- net /C8: track 239.8 -> 24.2 mm, vias 3 -> 0
- net /C6: track 238.8 -> 24.7 mm, vias 3 -> 0
- net Net-(C9-Pad1): track 24.9 -> 234.3 mm, vias 0 -> 3
- net /GND1: track 217.6 -> 35.9 mm
- net Net-(C13-Pad2): track 15.1 -> 189.1 mm, vias 0 -> 3
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- added copper zone on In2.Cu, net /GND1
- added copper zone on B.Cu, net /VREG
- removed copper zone on In1.Cu, net /GND1
Other:
- board size 50 x 287 mm -> 50 x 236.2 mm
- board text added: "1_V0"
- board text added: "1_V1"
- board text added: "1_V2"
- board text added: "1_V3"
- board text added: "1_V4"
- board text added: "1_V5"
- board text added: "1_V6"
- board text added: "1_V7"
- board text added: "1_V8"
- board text added: "2_V0"
- board text added: "2_V1"
- board text added: "2_V2"
- board text added: "2_V3"
- board text added: "2_V4"
- board text added: "2_V5"
- board text added: "2_V6"
- board text added: "2_V7"
- board text added: "2_V8"
- board text added: "BMS Peripheral Rev 2.0 Olin Electric Motorsports Corey Cochran-Lepiz 2/27/2019"
- board text added: "Balancing Gate Resistors"
- board text added: "GND1"
- board text added: "GND2"
- board text added: "ID:"
- board text added: "IMA1"
- board text added: "IMA2"
- board text added: "IMB1"
- board text added: "IMB2"
- board text added: "IPA1"
- board text added: "IPA2"
- board text added: "IPB1"
- board text added: "IPB2"
- board text added: "Iso-SPI Towads Core"
- board text added: "Iso-SPI Up Daisy Chain"
- board text added: "Sense Resistors"
- board text added: "Temp Resistors"
- board text added: "Tented vias for GND here?"
- board text added: "V2"
- board text added: "VREG"
- board text removed: "BMS Peripheral Rev 1.1 Olin Electric Motorsports Corey Cochran-Lepiz"
